File: formant_vco.kicad_pcb (KiCad board)
At the start: 2 copper layers, 20 x 128.5 mm, 80 parts, among them J1 JACK_2P, J2 JACK_2P, J3 JACK_2P, J4 CONN_01X03, J5 JACK_2P, Q1 BC850, Q2 BC850, Q3 BC850, Q4 BC850, Q5 BC850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

Commit message: Add footprints for mono jack and alpha pots
Parts:
- removed REF** (x2): MountingHole_6.4mm_M6, Mounting_Holes:MountingHole_6.4mm_M6
- removed REF** (x2): MountingHole_3.2mm_M3, Mounting_Holes:MountingHole_3.2mm_M3
- removed U4: 7805, TO_SOT_Packages_SMD:SOT-23
- added D3, D4: LED, LEDs:LED_D5.0mm, F.Cu at (0.00, 0.00)
- added R31: 100K, Resistors_SMD:R_0603, F.Cu at (204.0, 50.6)
- added R32: 1K, Resistors_SMD:R_0603, F.Cu at (207.2, 61.9)
- added SW2: SWITCH_SPST, Pin_Headers:Pin_Header_Straight_2x01_Pitch2.54mm, F.Cu at (154.3, 72.9)
- C1, C12, C13, C15, C16, C2, C4: footprint Capacitors_Tantalum_SMD:CP_Tantalum_Case-A_EIA-3216-18_Hand -> Capacitors_Tantalum_SMD:CP_Tantalum_Case-A_EIA-3216-18_Reflow
- J4: value CONN_01X03 -> CONN_02X08; footprint Pin_Headers:Pin_Header_Straight_1x03_Pitch2.54mm -> Connectors:IDC_Header_Straight_16pins
- RV1, RV2, RV3, RV4: footprint Potentiometers:Potentiometer_Bourns_PTV09A-1_Horizontal -> footprint_alpha_d_pot:alpha_d_pot_vert
- moved J4 199.9 mm to (0.00, 0.00)
- moved C17 121.7 mm to (217.6, 29.1), turned to 0 degrees
- moved J5 118.7 mm to (190.5, 30.0)
- moved R9 117.9 mm to (213.2, 41.6), turned to 0 degrees
- moved Q1 116.8 mm to (205.0, 37.3), turned to 0 degrees
- moved C8 111.3 mm to (221.7, 29.1)
- moved RV4 110.1 mm to (167.0, 37.8), turned to 0 degrees
- moved RV8 102.7 mm to (195.9, 30.8), turned to 0 degrees
- moved R27 101.7 mm to (222.0, 39.4), turned to 0 degrees
- moved R18 101.7 mm to (220.6, 44.4), turned to 0 degrees
- moved C2 99.0 mm to (211.4, 30.2)
- moved R25 97.6 mm to (204.0, 55.6), turned to 0 degrees
- moved C6 97.2 mm to (209.7, 41.6), turned to 0 degrees
- moved J3 94.6 mm to (162.0, 60.1), turned to 0 degrees
- moved D1 93.9 mm to (210.7, 36.4), turned to 0 degrees
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Connections:
- C10 pad 1: GND -> Net-(C10-Pad1)
- C11 pad 2: GND -> Net-(C10-Pad1)
- C12 pad 2: GND -> Net-(C10-Pad1)
- C13 pad 1: GND -> Net-(C10-Pad1)
- C15 pad 2: GND -> Net-(C10-Pad1)
- C16 pad 1: GND -> Net-(C10-Pad1)
- C4 pad 1: +5V -> Net-(C4-Pad1)
- C5 pad 2: +5V -> Net-(C4-Pad1)
- C6 pad 1: GND -> Net-(C10-Pad1)
- C7 pad 2: GND -> Net-(C10-Pad1)
- C8 pad 1: GND -> Net-(C10-Pad1)
- C9 pad 2: GND -> Net-(C10-Pad1)
- J4 pad 1: +15V -> -15V
- J4 pad 2: GND -> -15V
- J4 pad 3: -15V -> GND
- U1 pad 1: Net-(U1-Pad1) -> (no net)
- U1 pad 3: Net-(U1-Pad3) -> (no net)
- U1 pad 5: Net-(U1-Pad5) -> (no net)
- U1 pad 7: Net-(U1-Pad7) -> (no net)
- U3 pad 10: Net-(U3-Pad10) -> (no net)
- U3 pad 11: Net-(U3-Pad11) -> (no net)
- U3 pad 12: Net-(U3-Pad12) -> (no net)
- U3 pad 13: Net-(U3-Pad13) -> (no net)
- U3 pad 4: Net-(U3-Pad4) -> (no net)
- U3 pad 5: Net-(U3-Pad5) -> (no net)
- U3 pad 6: Net-(U3-Pad6) -> (no net)
- U3 pad 8: Net-(U3-Pad8) -> (no net)
- U3 pad 9: Net-(U3-Pad9) -> (no net)
- U5 pad 1: Net-(U5-Pad1) -> Net-(R32-Pad2)
- U5 pad 2: Net-(U5-Pad2) -> Net-(R32-Pad2)
- U5 pad 3: Net-(U5-Pad3) -> Net-(C17-Pad2)
- U5 pad 5: Net-(U5-Pad5) -> (no net)
- U5 pad 6: Net-(U5-Pad6) -> (no net)
- U5 pad 7: Net-(U5-Pad7) -> (no net)
Routing:
- net +15V: track 115.8 -> 0.00 mm, vias 8 -> 0
- net +5V: track 115.6 -> 0.00 mm, vias 10 -> 0
- net Net-(R12-Pad2): track 105.5 -> 0.00 mm, vias 2 -> 0
- net +10V_REF: track 101.0 -> 0.00 mm, vias 4 -> 0
- net -15V: track 94.8 -> 0.00 mm, vias 7 -> 0
- net -10V_REF: track 76.9 -> 0.00 mm, vias 2 -> 0
- net GND: track 70.3 -> 0.00 mm, vias 27 -> 0
- net Net-(RV6-Pad3): track 59.5 -> 0.00 mm, vias 7 -> 0
- net SYNC_IN: track 51.8 -> 0.00 mm, vias 4 -> 0
- net Net-(R21-Pad1): track 44.5 -> 0.00 mm, vias 2 -> 0
- net Net-(C18-Pad1): track 38.0 -> 0.00 mm, vias 2 -> 0
- net Net-(C14-Pad1): track 35.7 -> 0.00 mm, vias 2 -> 0
- net Net-(Q5-Pad2): track 31.1 -> 0.00 mm, vias 2 -> 0
- net Net-(C3-Pad2): track 23.5 -> 0.00 mm, vias 2 -> 0
- net Net-(D1-Pad2): track 23.5 -> 0.00 mm, vias 2 -> 0
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- removed copper zone on B.Cu, net GND
- removed copper zone on F.Cu, net GND
Other:
- board outline removed
- rule pad_to_mask_clearance: 0.2 -> 0

Commit message: Start placing things
Parts:
- added U4: TL072, Housings_SOIC:SOIC-8_3.9x4.9mm_Pitch1.27mm, F.Cu at (163.3, 38.0)
- added U7: TL072, Housings_SOIC:SOIC-8_3.9x4.9mm_Pitch1.27mm, F.Cu at (77.3, 70.0)
- added ~: MountingHole_3.2mm_M3, Mounting_Holes:MountingHole_3.2mm_M3, F.Cu at (63.4, 172.3)
- added ~: MountingHole_3.2mm_M3, Mounting_Holes:MountingHole_3.2mm_M3, F.Cu at (63.4, 49.8)
- added ~: MountingHole_3.2mm_M3, Mounting_Holes:MountingHole_3.2mm_M3, F.Cu at (88.8, 49.8)
- added ~: MountingHole_3.2mm_M3, Mounting_Holes:MountingHole_3.2mm_M3, F.Cu at (88.8, 172.3)
- J1, J2, J3: footprint Pin_Headers:Pin_Header_Straight_1x03_Pitch2.54mm -> footprint_pj3010bm:pj301bm
- J5: footprint Socket_Strips:Socket_Strip_Straight_1x03_Pitch2.54mm -> footprint_pj3010bm:pj301bm
- U2, U5: value TL074 -> TL072; footprint Housings_SOIC:SOIC-14_3.9x8.7mm_Pitch1.27mm -> Housings_SOIC:SOIC-8_3.9x4.9mm_Pitch1.27mm
- moved J4 184.9 mm to (92.3, 160.3), turned to 90 degrees
- moved C17 181.9 mm to (73.3, 139.8), turned to 270 degrees
- moved J5 175.4 mm to (76.8, 163.5)
- moved D3 170.5 mm to (79.3, 151.0)
- moved R2 169.1 mm to (61.8, 88.5)
- moved RV8 167.9 mm to (70.0, 142.0)
- moved D4 167.2 mm to (71.8, 151.0)
- moved R32 160.7 mm to (70.5, 146.3), turned to 90 degrees
- moved R25 156.7 mm to (83.3, 155.5), turned to 180 degrees
- moved R9 153.8 mm to (87.8, 130.5), turned to 180 degrees
- moved R11 148.1 mm to (72.8, 68.5), turned to 270 degrees
- moved R5 146.6 mm to (67.8, 70.5), turned to 180 degrees
- moved Q1 145.6 mm to (92.3, 129.5), turned to 90 degrees
- moved R6 140.1 mm to (78.3, 60.0)
- moved J2 138.2 mm to (66.8, 103.5)
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Connections:
- U2 pad 1: -10V_REF -> Net-(R12-Pad1)
- U2 pad 2: Net-(R11-Pad2) -> Net-(R12-Pad2)
- U2 pad 4: +15V -> -15V
- U2 pad 5: Net-(RV6-Pad3) -> GND
- U2 pad 6: Net-(R13-Pad2) -> Net-(C3-Pad2)
- U2 pad 7: Net-(R13-Pad2) -> Net-(C3-Pad1)
- U2 pad 8: Net-(R12-Pad1) -> +15V
- U5 pad 1: Net-(R32-Pad2) -> Net-(C17-Pad2)
- U5 pad 2: Net-(R32-Pad2) -> Net-(C17-Pad1)
- U5 pad 3: Net-(C17-Pad2) -> Net-(RV6-Pad3)
- U5 pad 4: +15V -> -15V
- U5 pad 5: (no net) -> Net-(C17-Pad2)
- U5 pad 6: (no net) -> Net-(R32-Pad2)
- U5 pad 7: (no net) -> Net-(R32-Pad2)
- U5 pad 8: Net-(C17-Pad2) -> +15V
Routing:
- added copper zone on B.Cu, net GND
- added copper zone on F.Cu, net GND
Other:
- board outline added: 65 x 128.5 mm

Commit message: place rest of components
Parts:
- moved C9 181.0 mm to (63.3, 149.0), turned to 270 degrees
- moved C16 167.9 mm to (65.8, 149.3), turned to 90 degrees
- moved C8 164.2 mm to (63.3, 142.3), turned to 270 degrees
- moved R18 157.4 mm to (66.0, 130.5), turned to 180 degrees
- moved C15 150.9 mm to (65.8, 142.3), turned to 90 degrees
- moved Q5 144.7 mm to (78.5, 104.3), turned to 90 degrees
- moved R19 144.4 mm to (72.3, 108.8), turned to 270 degrees
- moved R23 142.6 mm to (71.8, 110.8), turned to 180 degrees
- moved R21 141.1 mm to (71.8, 113.3), turned to 180 degrees
- moved R22 134.7 mm to (65.0, 110.8), turned to 180 degrees
- moved RV5 133.2 mm to (75.3, 88.8)
- moved R28 132.8 mm to (81.3, 111.5), turned to 270 degrees
- moved R17 131.9 mm to (68.5, 128.8)
- moved C5 131.5 mm to (82.0, 130.5)
- moved Q4 130.4 mm to (72.8, 134.0), turned to 180 degrees
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Connections:
- C4 pad 1: Net-(C4-Pad1) -> +5V
- C5 pad 2: Net-(C4-Pad1) -> +5V

Commit message: Some routing
Routing:
- net +10V_REF: track 0.00 -> 37.6 mm
- net Net-(R12-Pad2): track 0.00 -> 32.9 mm
- net Net-(C17-Pad2): track 0.00 -> 27.2 mm
- net -15V: track 0.00 -> 22.1 mm
- net Net-(D3-Pad2): track 0.00 -> 18.5 mm
- net +5V: track 0.00 -> 18.4 mm
- net +15V: track 0.00 -> 15.1 mm
- net Net-(C10-Pad1): track 0.00 -> 15.0 mm
- net Net-(J1-Pad1): track 0.00 -> 14.5 mm
- net Net-(J5-Pad1): track 0.00 -> 13.9 mm
- net GND: track 0.00 -> 12.4 mm
- net SYNC_IN: track 0.00 -> 8.67 mm
- net Net-(J3-Pad1): track 0.00 -> 8.10 mm
- net Net-(J2-Pad1): track 0.00 -> 8.10 mm
- net Net-(C14-Pad1): track 0.00 -> 6.84 mm
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Other:
- net class Default: trace_width 0.25 -> 0.4

Commit message: Final routing, fab outputs
Parts:
- removed ~ (x4): MountingHole_3.2mm_M3, Mounting_Holes:MountingHole_3.2mm_M3
Connections:
- C10 pad 1: Net-(C10-Pad1) -> GND
- C11 pad 2: Net-(C10-Pad1) -> GND
- C12 pad 2: Net-(C10-Pad1) -> GND
- C13 pad 1: Net-(C10-Pad1) -> GND
- C15 pad 2: Net-(C10-Pad1) -> GND
- C16 pad 1: Net-(C10-Pad1) -> GND
- C6 pad 1: Net-(C10-Pad1) -> GND
- C7 pad 2: Net-(C10-Pad1) -> GND
- C8 pad 1: Net-(C10-Pad1) -> GND
- C9 pad 2: Net-(C10-Pad1) -> GND
Routing:
- net +15V: track 15.1 -> 167.3 mm, vias 0 -> 11
- net -15V: track 22.1 -> 150.3 mm, vias 0 -> 8
- net GND: track 12.4 -> 124.7 mm, vias 0 -> 13
- net CV_BUS: track 0.00 -> 88.4 mm
- net Net-(RV6-Pad3): track 0.00 -> 77.2 mm, vias 0 -> 6
- net Net-(R12-Pad2): track 32.9 -> 104.4 mm, vias 0 -> 4
- net +5V: track 18.4 -> 77.3 mm, vias 0 -> 4
- net Net-(C18-Pad1): track 0.00 -> 53.7 mm, vias 0 -> 6
- net Net-(C18-Pad2): track 1.60 -> 51.9 mm, vias 0 -> 4
- net -10V_REF: track 5.75 -> 53.3 mm, vias 0 -> 2
- net +10V_REF: track 37.6 -> 79.5 mm, vias 0 -> 2
- net Net-(C3-Pad2): track 2.13 -> 41.9 mm, vias 0 -> 6
- net Net-(RV5-Pad2): track 0.00 -> 32.8 mm, vias 0 -> 2
- net Net-(J3-Pad1): track 8.10 -> 36.9 mm
- net Net-(J2-Pad1): track 8.10 -> 36.2 mm, vias 0 -> 2
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Other:
- board size 65 x 128.5 mm -> 39.8 x 110.4 mm
- board text added: "AF VCO REV. 1A"
- board text added: "sebholzapfel.com 2017"
