File: formant_vco.sch (KiCad schematic (older format))
At the start: 81 parts, among them J1 JACK_2P, J2 JACK_2P, J3 JACK_2P, J4 CONN_02X08, J5 JACK_2P, Q1 BC850, Q2 BC850, Q3 BC850, Q4 BC850, Q5 BC850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

Commit message: Start placing things
Parts:
- added U7: TL072, Housings_SOIC:SOIC-8_3.9x4.9mm_Pitch1.27mm, symbol TL072
- renumbered U4 to U2, U5 to U4, U2 to U4, U4 to U5
Connections:
- net +15V: now also U7.8 (V+)
- net -10V_REF: now also U7.1
- net -15V: now also U7.4 (V-)
- net GND: now also U2.3 (+), U2.5 (+), U7.3 (+); no longer U2.3 (+), U2.5 (+)
- net at R11.2, R3.1: now also U7.2 (-)
- net at R12.2, R31.1, R4.1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: now also U2.2 (-); no longer U2.6 (-)
- net at R12.1, RV5.1: now also U2.1; no longer U2.7
- net at C3.2, R15.1, U6.1: now also U2.6 (-); no longer U2.2 (-)
- net at C3.1, R19.1: now also U2.7; no longer U2.1
- net at C18.1, RV7.2: now also U4.6 (-); no longer U4.2 (-)
- net at C18.2, R26.1: now also U4.7; no longer U4.1
- net at R21.1, U6.6, U6.8: now also U4.5 (+); no longer U4.3 (+)
- net at RV6.3, U4.3 (+), U6.5: now also U5.3 (+); no longer U5.5 (+)
- net at C17.1, R24.1, RV9.3: now also U5.2 (-); no longer U5.6 (-)
- net at C17.2, R25.1, RV9.1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: now also U5.1; no longer U5.7
Other:
- moved on the sheet: U3B, U3C, U3D
Changed lines of the file:
@@
 L CD4093 U3
 U 2 1 5962EB92
-P 4750 6725
-F 0 "U3" H 4850 6825 60  0000 C CNN
-F 1 "CD4093" H 4950 6550 60  0000 C CNN
-F 2 "Housings_SOIC:SOIC-14_3.9x8.7mm_Pitch1.27mm" H 4800 6625 60  0001 C CNN
-F 3 "" H 4800 6625 60  0001 C CNN
-	2    4750 6725
+P 6300 6600
+F 0 "U3" H 6400 6700 60  0000 C CNN
+F 1 "CD4093" H 6500 6425 60  0000 C CNN
+F 2 "Housings_SOIC:SOIC-14_3.9x8.7mm_Pitch1.27mm" H 6350 6500 60  0001 C CNN
+F 3 "" H 6350 6500 60  0001 C CNN
+	2    6300 6600
 	1    0    0    -1
 $EndComp
@@
 L CD4093 U3
 U 3 1 5962EC6B
-P 4650 7000
-F 0 "U3" H 4750 7100 60  0000 C CNN
-F 1 "CD4093" H 4850 6825 60  0000 C CNN
-F 2 "Housings_SOIC:SOIC-14_3.9x8.7mm_Pitch1.27mm" H 4700 6900 60  0001 C CNN
-F 3 "" H 4700 6900 60  0001 C CNN
-	3    4650 7000
+P 6200 6875
+F 0 "U3" H 6300 6975 60  0000 C CNN
+F 1 "CD4093" H 6400 6700 60  0000 C CNN
+F 2 "Housings_SOIC:SOIC-14_3.9x8.7mm_Pitch1.27mm" H 6250 6775 60  0001 C CNN
+F 3 "" H 6250 6775 60  0001 C CNN
+	3    6200 6875
 	1    0    0    -1
 $EndComp
@@
 L CD4093 U3
 U 4 1 5962ED4E
-P 4600 7250
-F 0 "U3" H 4700 7350 60  0000 C CNN
-F 1 "CD4093" H 4800 7075 60  0000 C CNN
-F 2 "Housings_SOIC:SOIC-14_3.9x8.7mm_Pitch1.27mm" H 4650 7150 60  0001 C CNN
-F 3 "" H 4650 7150 60  0001 C CNN
-	4    4600 7250
+P 6150 7125
+F 0 "U3" H 6250 7225 60  0000 C CNN
+F 1 "CD4093" H 6350 6950 60  0000 C CNN
+F 2 "Housings_SOIC:SOIC-14_3.9x8.7mm_Pitch1.27mm" H 6200 7025 60  0001 C CNN
+F 3 "" H 6200 7025 60  0001 C CNN
+	4    6150 7125
 	1    0    0    -1
 $EndComp
@@
 $Comp
 L TL072 U2
-U 2 1 596B241F
+U 1 1 596B241F
 P 4200 4500
 F 0 "U2" H 4200 4700 50  0000 L CNN
@@
 F 2 "Housings_SOIC:SOIC-8_3.9x4.9mm_Pitch1.27mm" H 4200 4500 50  0001 C CNN
 F 3 "" H 4200 4500 50  0001 C CNN
-	2    4200 4500
+	1    4200 4500
 	1    0    0    1
 $EndComp
 $Comp
-L TL072 U4
-U 1 1 596B2732
+L TL072 U2
+U 2 1 596B2732
 P 5500 5200
-F 0 "U4" H 5500 5400 50  0000 L CNN
+F 0 "U2" H 5500 5400 50  0000 L CNN
 F 1 "TL072" H 5500 5000 50  0000 L CNN
 F 2 "Housings_SOIC:SOIC-8_3.9x4.9mm_Pitch1.27mm" H 5500 5200 50  0001 C CNN
 F 3 "" H 5500 5200 50  0001 C CNN
-	1    5500 5200
+	2    5500 5200
 	1    0    0    1
 $EndComp
 $Comp
-L TL072 U5
-U 1 1 596B288E
+L TL072 U4
+U 2 1 596B288E
 P 9150 4550
-F 0 "U5" H 9150 4750 50  0000 L CNN
+F 0 "U4" H 9150 4750 50  0000 L CNN
 F 1 "TL072" H 9150 4350 50  0000 L CNN
 F 2 "Housings_SOIC:SOIC-8_3.9x4.9mm_Pitch1.27mm" H 9150 4550 50  0001 C CNN
 F 3 "" H 9150 4550 50  0001 C CNN
-	1    9150 4550
+	2    9150 4550
 	1    0    0    1
 $EndComp
 $Comp
-L TL072 U4
-U 2 1 596B30CA
+L TL072 U5
+U 1 1 596B30CA
 P 8900 3050
-F 0 "U4" H 8900 3250 50  0000 L CNN
+F 0 "U5" H 8900 3250 50  0000 L CNN
 F 1 "TL072" H 8900 2850 50  0000 L CNN
 F 2 "Housings_SOIC:SOIC-8_3.9x4.9mm_Pitch1.27mm" H 8900 3050 50  0001 C CNN
 F 3 "" H 8900 3050 50  0001 C CNN
-	2    8900 3050
+	1    8900 3050
 	1    0    0    1
 $EndComp
 $Comp
-L TL072 U2
+L TL072 U4
 U 1 1 596B34D6
 P 3800 2350
-F 0 "U2" H 3800 2550 50  0000 L CNN
+F 0 "U4" H 3800 2550 50  0000 L CNN
 F 1 "TL072" H 3800 2150 50  0000 L CNN
 F 2 "Housings_SOIC:SOIC-8_3.9x4.9mm_Pitch1.27mm" H 3800 2350 50  0001 C CNN
@@
 	1    0    0    -1
 $EndComp
+$Comp
+L TL072 U7
+U 1 1 596C40BF
+P 2750 1500
+F 0 "U7" H 2750 1700 50  0000 L CNN
+F 1 "TL072" H 2750 1300 50  0000 L CNN
+F 2 "Housings_SOIC:SOIC-8_3.9x4.9mm_Pitch1.27mm" H 2750 1500 50  0001 C CNN
+F 3 "" H 2750 1500 50  0001 C CNN
+	1    2750 1500
+	1    0    0    1
+$EndComp
 $EndSCHEMATC

Commit message: place rest of components
Connections:
- net +5V: now also C4.1, C5.2
Changed lines of the file:
@@
 	1    0    0    1
 $EndComp
+Connection ~ 6200 925
 $EndSCHEMATC

Commit message: Final routing, fab outputs
Connections:
- net GND: now also C10.1, C11.2, C12.2, C13.1, C15.2, C16.1, C6.1, C7.2, C8.1, C9.2
Changed lines of the file:
@@
 L GND #PWR035
 U 1 1 5965232A
-P 7775 1000
-F 0 "#PWR035" H 7775 750 50  0001 C CNN
-F 1 "GND" H 7775 850 50  0000 C CNN
-F 2 "" H 7775 1000 50  0001 C CNN
-F 3 "" H 7775 1000 50  0001 C CNN
-	1    7775 1000
+P 7750 1000
+F 0 "#PWR035" H 7750 750 50  0001 C CNN
+F 1 "GND" H 7750 850 50  0000 C CNN
+F 2 "" H 7750 1000 50  0001 C CNN
+F 3 "" H 7750 1000 50  0001 C CNN
+	1    7750 1000
 	0    -1   -1   0
 $EndComp
